File: PCB/heating.kicad_pcb (KiCad board)
At the start: 2 copper layers, 72.4 x 100.3 mm, 23 parts, among them J1 Conn_01x02_Male, J10 Conn_01x04_Male, J11 Conn_01x02_Male, J12 Conn_01x03_Male, J13 Conn_01x03_Male, J14 Conn_01x03_Male, J15 Conn_01x02_Male, J2 Conn_01x04_Male, J3 Conn_01x04_Male, J4 Conn_01x02_Male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

Commit message: Update PCB Layout
Parts:
- A1: moved to B.Cu
- R1, R2, R3, R4, R5: footprint Resistor_THT:R_Axial_DIN0414_L11.9mm_D4.5mm_P20.32mm_Horizontal -> Resistor_THT:R_Axial_DIN0411_L9.9mm_D3.6mm_P12.70mm_Horizontal
- moved J4 76.7 mm to (180.3, 57.1), turned to 90 degrees
- moved J13 75.0 mm to (171.4, 121.9), turned to 270 degrees
- moved R5 75.0 mm to (144.8, 54.6)
- moved J14 74.9 mm to (176.5, 121.9), turned to 270 degrees
- moved J1 59.5 mm to (143.5, 120.7), turned to 90 degrees
- moved J11 59.0 mm to (181.6, 100.3), turned to 90 degrees
- moved A1 58.5 mm to (143.5, 111.8)
- moved J8 56.8 mm to (156.2, 54.6), turned to 180 degrees
- moved R4 56.1 mm to (162.6, 54.6), turned to 90 degrees
- moved R3 56.0 mm to (166.4, 54.6), turned to 90 degrees
- moved R2 55.9 mm to (170.2, 54.6), turned to 90 degrees
- moved R1 55.8 mm to (166.4, 118.1)
- moved J12 55.5 mm to (168.9, 100.3)
- moved C1 54.7 mm to (137.2, 97.8)
- moved J5 48.3 mm to (180.3, 72.4)
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Routing:
- net Net-(A1-Pad27): track 93.5 -> 14.1 mm, vias 2 -> 0
- net GND: track 368.6 -> 306.0 mm
- net Net-(A1-Pad26): track 62.7 -> 14.1 mm, vias 2 -> 0
- net Net-(A1-Pad23): track 58.0 -> 14.6 mm, vias 2 -> 0
- net Net-(A1-Pad24): track 44.7 -> 14.6 mm, vias 2 -> 0
- net +3V3: track 57.5 -> 86.1 mm
- net Net-(A1-Pad25): track 42.4 -> 14.6 mm, vias 2 -> 0
- net Net-(J2-Pad3): track 29.6 -> 5.24 mm
- net Net-(A1-Pad17): track 30.3 -> 10.2 mm
- net Net-(A1-Pad8): track 11.0 -> 28.8 mm, vias 0 -> 2
- net Net-(A1-Pad28): track 41.8 -> 24.5 mm, vias 2 -> 0
- net Net-(A1-Pad19): track 35.7 -> 20.6 mm
- net Net-(A1-Pad10): track 26.0 -> 11.4 mm
- net Net-(A1-Pad9): track 19.6 -> 31.3 mm, vias 0 -> 2
- net Net-(A1-Pad18): track 15.6 -> 6.92 mm
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Other:
- board size 72.4 x 100.3 mm -> 76.2 x 100.3 mm

Commit message: Update PCB
Parts:
- R1: value 10k -> 100k
Changed lines of the file:
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@@
   )
   (setup
-    (last_trace_width 1)
+    (last_trace_width 0.25)
     (user_trace_width 1)
     (trace_clearance 0.2)
@@
       (effects (font (size 1 1) (thickness 0.15)))
     )
-    (fp_text value 10k (at 6.35 2.92 90) (layer F.Fab)
+    (fp_text value 100k (at 6.35 2.92 90) (layer F.Fab)
       (effects (font (size 1 1) (thickness 0.15)))
     )
@@
   (gr_line (start 187.96 46.99) (end 187.96 134.62) (layer F.SilkS) (width 0.12))
   (gr_line (start 111.76 46.99) (end 187.96 46.99) (layer F.SilkS) (width 0.12))
-  (via (at 184.15 62.23) (size 2) (drill 1) (layers F.Cu B.Cu) (net 20))
-  (via (at 181.61 90.17) (size 2) (drill 1) (layers F.Cu B.Cu) (net 20))
   (segment (start 123.77 71.12) (end 126.31 68.58) (width 1) (layer F.Cu) (net 5))
   (segment (start 121.92 71.12) (end 123.77 71.12) (width 1) (layer F.Cu) (net 5))
@@
   (segment (start 163.83 58.42) (end 163.83 63.5) (width 1) (layer F.Cu) (net 19))
   (segment (start 156.17 54.61) (end 162.56 54.61) (width 1) (layer F.Cu) (net 19))
+  (via (at 184.15 62.23) (size 2) (drill 1) (layers F.Cu B.Cu) (net 20))
+  (via (at 181.61 90.17) (size 2) (drill 1) (layers F.Cu B.Cu) (net 20))
   (segment (start 144.78 77.47) (end 144.78 78.74) (width 1) (layer F.Cu) (net 20))
   (segment (start 144.78 78.74) (end 142.24 81.28) (width 1) (layer F.Cu) (net 20))
