File: PCB/heating.sch (KiCad schematic (older format))
At the start: 23 parts, among them J1 Conn_01x02_Male, J10 Conn_01x04_Male, J11 Conn_01x02_Male, J12 Conn_01x03_Male, J13 Conn_01x03_Male, J14 Conn_01x03_Male, J15 Conn_01x02_Male, J2 Conn_01x04_Male, J3 Conn_01x04_Male, J4 Conn_01x02_Male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

Commit message: Update PCB Layout
Parts:
- R1, R2, R3, R4, R5: footprint Resistor_THT:R_Axial_DIN0414_L11.9mm_D4.5mm_P20.32mm_Horizontal -> Resistor_THT:R_Axial_DIN0411_L9.9mm_D3.6mm_P12.70mm_Horizontal
Changed lines of the file:
@@
 F 0 "R1" H 1120 1446 50  0000 L CNN
 F 1 "10k" H 1120 1355 50  0000 L CNN
-F 2 "Resistor_THT:R_Axial_DIN0414_L11.9mm_D4.5mm_P20.32mm_Horizontal" V 980 1400 50  0001 C CNN
+F 2 "Resistor_THT:R_Axial_DIN0411_L9.9mm_D3.6mm_P12.70mm_Horizontal" V 980 1400 50  0001 C CNN
 F 3 "~" H 1050 1400 50  0001 C CNN
 	1    1050 1400
@@
 F 0 "R2" H 1120 2646 50  0000 L CNN
 F 1 "10k" H 1120 2555 50  0000 L CNN
-F 2 "Resistor_THT:R_Axial_DIN0414_L11.9mm_D4.5mm_P20.32mm_Horizontal" V 980 2600 50  0001 C CNN
+F 2 "Resistor_THT:R_Axial_DIN0411_L9.9mm_D3.6mm_P12.70mm_Horizontal" V 980 2600 50  0001 C CNN
 F 3 "~" H 1050 2600 50  0001 C CNN
 	1    1050 2600
@@
 F 0 "R3" H 2820 3696 50  0000 L CNN
 F 1 "10k" H 2820 3605 50  0000 L CNN
-F 2 "Resistor_THT:R_Axial_DIN0414_L11.9mm_D4.5mm_P20.32mm_Horizontal" V 2680 3650 50  0001 C CNN
+F 2 "Resistor_THT:R_Axial_DIN0411_L9.9mm_D3.6mm_P12.70mm_Horizontal" V 2680 3650 50  0001 C CNN
 F 3 "~" H 2750 3650 50  0001 C CNN
 	1    2750 3650
@@
 F 0 "R4" H 3570 3696 50  0000 L CNN
 F 1 "10k" H 3570 3605 50  0000 L CNN
-F 2 "Resistor_THT:R_Axial_DIN0414_L11.9mm_D4.5mm_P20.32mm_Horizontal" V 3430 3650 50  0001 C CNN
+F 2 "Resistor_THT:R_Axial_DIN0411_L9.9mm_D3.6mm_P12.70mm_Horizontal" V 3430 3650 50  0001 C CNN
 F 3 "~" H 3500 3650 50  0001 C CNN
 	1    3500 3650
@@
 F 0 "R5" H 3970 4646 50  0000 L CNN
 F 1 "10k" H 3970 4555 50  0000 L CNN
-F 2 "Resistor_THT:R_Axial_DIN0414_L11.9mm_D4.5mm_P20.32mm_Horizontal" V 3830 4600 50  0001 C CNN
+F 2 "Resistor_THT:R_Axial_DIN0411_L9.9mm_D3.6mm_P12.70mm_Horizontal" V 3830 4600 50  0001 C CNN
 F 3 "~" H 3900 4600 50  0001 C CNN
 	1    3900 4600

Commit message: Update PCB
Parts:
- R1: value 10k -> 100k
Changed lines of the file:
@@
 P 1050 1400
 F 0 "R1" H 1120 1446 50  0000 L CNN
-F 1 "10k" H 1120 1355 50  0000 L CNN
+F 1 "100k" H 1120 1355 50  0000 L CNN
 F 2 "Resistor_THT:R_Axial_DIN0411_L9.9mm_D3.6mm_P12.70mm_Horizontal" V 980 1400 50  0001 C CNN
 F 3 "~" H 1050 1400 50  0001 C CNN
